Commit message: Fix sleep pose for the Locobot

File: interbotix_ros_xsarms/interbotix_xsarm_moveit/config/srdf/wx200.srdf.xacro (robot description, xacro)
@@ -47,5 +47,5 @@
     <group_state name="Sleep" group="interbotix_arm">
         <joint name="elbow" value="1.55" />
-        <joint name="shoulder" value="-1.88" />
+        <joint name="shoulder" value="-1.35" />
         <joint name="waist" value="0" />
         <joint name="wrist_angle" value="0.8" />
